File: v1.2/Eagle/LumaFix64v1.2_sp.sch (EAGLE design)
At the start: 11 parts, among them IC1 74HCT14D

Commit message: Silk Screen Update
Parts:
- added U$13: OPEN_SOURCE_HW, Logo:OPEN_SOURCE_HW
Other:
- note added: "http://github.com/svenpetersen1965"
Changed lines of the file:
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@@
 <layer number="250" name="Descript" color="7" fill="1" visible="no" active="no"/>
 <layer number="251" name="SMDround" color="7" fill="1" visible="no" active="no"/>
+<layer number="252" name="BR-BS" color="7" fill="1" visible="no" active="yes"/>
+<layer number="253" name="BR-LS" color="7" fill="1" visible="no" active="yes"/>
 <layer number="254" name="OrgLBR" color="7" fill="1" visible="no" active="no"/>
 <layer number="255" name="Accent" color="7" fill="1" visible="yes" active="yes"/>
@@
 <part name="CP1" library="Cutpad" deviceset="OPEN" device=""/>
 <part name="R1" library="SMD" deviceset="R-0805" device="" value="n/a"/>
+<part name="U$13" library="Logo" deviceset="OPEN_SOURCE_HW" device=""/>
 </parts>
 <sheets>
@@
 desired and CHR pot
 not populated.</text>
+<text x="170.18" y="7.62" size="2.54" layer="95">http://github.com/svenpetersen1965</text>
 </plain>
 <instances>
@@
 <attribute name="VALUE" x="91.44" y="34.29" size="1.27" layer="96" ratio="10"/>
 </instance>
+<instance part="U$13" gate="G$1" x="129.54" y="7.62" smashed="yes"/>
 </instances>
 <busses>
